File: eagle/untitled.sch (EAGLE design)
At the start: 47 parts, among them J1 JTAG, Q1 16MHz, U1 MMA3202KEG

Commit message: Update board.
Parts:
- removed D11: DIODE, gipi:DIODE
- removed G1: BAT, SparkFun-Electromechanical:BATTERY20PTH
- added C7, C8, C9: 10nF, SparkFun-Capacitors:CAP0603-CAP
- added D13: (no value), diode:SCHOTTKY-DIODESMD
- added JP6: M02JST-PTH-VERT, SparkFun-Connectors:M02JST-PTH-VERT
- added L1: (no value), SparkFun-Passives:INDUCTOR0603
- added LED1: (no value), SparkFun-LED:LED0603
- added R16, R17, R18: 1k, SparkFun-Passives:RESISTOR0603-RES
- added U$3: V_REG_TPS61040SMD, SparkFun-PowerIC:V_REG_TPS61040SMD
- C1, C2, C3: device SparkFun-Capacitors:CAP1206 -> SparkFun-Capacitors:CAP0603-CAP
- C4, C5: value 10pF -> 10nF; device SparkFun-Capacitors:CAP1206 -> SparkFun-Capacitors:CAP0603-CAP
- GOLD_ORB_SM1: value OSHWLOGO_GOLD_ORB_SM -> OSHWLOGO_GOLD_ORB_LG; device bfl:OSHWLOGO_GOLD_ORB_SM -> bfl:OSHWLOGO_GOLD_ORB_LG
- JP1: value M11PTH -> M13; device SparkFun-Connectors:M11PTH -> SparkFun-Connectors:M13
- R10, R3, R9: device SparkFun-Passives:RESISTOR1206 -> SparkFun-Passives:RESISTOR0603-RES
Connections:
- removed net N$33: D11.A, G1.-
- new net GN: C4.1, C5.1, C6.2, D1.C, D2.C, D3.C, D4.C, D5.C, D6.C, D7.C, D8.C, D9.C, J1.10, J1.2, JP1.12, JP5.6, LED1.C, S1.1, S1.2, S2.3
- new net N$35: R16.1, U1.STATUS
- new net N$36: LED1.A, R16.2
- new net N$38: C7.2, JP6.1, L1.1, U$3.EN, U$3.VIN
- new net N$39: D13.A, L1.2, U$3.SW
- new net N$41: C8.1, R17.1, R18.2, U$3.FB
- new net N$42: C8.2, C9.2, D13.C, R17.2
- net GND-ISO: now also C7.1, C9.1, JP6.2, R18.1, U$3.GND; no longer C4.1, C5.1, C6.2, D1.C, D2.C, D3.C, D4.C, D5.C, D6.C, D7.C, D8.C, D9.C, G1.+, J1.10, J1.2, JP5.6, S1.1, S1.2, S2.3
- net N$28: no longer D11.C
- net VCC1: now also JP1.13
Other:
- moved on the sheet: C3
