File: eagle/untitled.sch (EAGLE design)
At the start: 56 parts, among them J1 JTAG, Q1 16MHz, U1 MMA3202KEG

Commit message: Add reverse voltage protection by P-MOSFET + Labelling.
Parts:
- added NFET: P-CHANNEL-MOSFET, GeekAmmo:P-CHANNEL-MOSFET
- renumbered U$3 to BOOST
Connections:
- new net N$33: JP6.1, NFET.S
- net GND-ISO: now also NFET.G
- net N$38: now also NFET.D; no longer JP6.1

Commit message: Rework labels.
Parts:
- D13: value (none) -> DIODE; device diode:SCHOTTKY-DIODESMD -> gipi:DIODE
Changed lines of the file:
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@@
 <grid distance="0.1" unitdist="inch" unit="inch" style="lines" multiple="1" display="no" altdistance="0.01" altunitdist="inch" altunit="inch"/>
 <layers>
-<layer number="1" name="Top" color="4" fill="1" visible="no" active="no"/>
-<layer number="16" name="Bottom" color="1" fill="1" visible="no" active="no"/>
-<layer number="17" name="Pads" color="2" fill="1" visible="no" active="no"/>
-<layer number="18" name="Vias" color="2" fill="1" visible="no" active="no"/>
-<layer number="19" name="Unrouted" color="2" fill="1" visible="no" active="no"/>
-<layer number="20" name="Dimension" color="15" fill="1" visible="no" active="no"/>
-<layer number="21" name="tPlace" color="7" fill="1" visible="no" active="no"/>
-<layer number="22" name="bPlace" color="15" fill="1" visible="no" active="no"/>
-<layer number="23" name="tOrigins" color="15" fill="1" visible="no" active="no"/>
-<layer number="24" name="bOrigins" color="15" fill="1" visible="no" active="no"/>
-<layer number="25" name="tNames" color="7" fill="1" visible="no" active="no"/>
-<layer number="26" name="bNames" color="7" fill="1" visible="no" active="no"/>
-<layer number="27" name="tValues" color="7" fill="1" visible="no" active="no"/>
-<layer number="28" name="bValues" color="7" fill="1" visible="no" active="no"/>
+<layer number="1" name="Top" color="4" fill="1" visible="yes" active="no"/>
+<layer number="16" name="Bottom" color="1" fill="1" visible="yes" active="no"/>
+<layer number="17" name="Pads" color="2" fill="1" visible="yes" active="no"/>
+<layer number="18" name="Vias" color="2" fill="1" visible="yes" active="no"/>
+<layer number="19" name="Unrouted" color="2" fill="1" visible="yes" active="no"/>
+<layer number="20" name="Dimension" color="15" fill="1" visible="yes" active="no"/>
+<layer number="21" name="tPlace" color="7" fill="1" visible="yes" active="no"/>
+<layer number="22" name="bPlace" color="15" fill="1" visible="yes" active="no"/>
+<layer number="23" name="tOrigins" color="15" fill="1" visible="yes" active="no"/>
+<layer number="24" name="bOrigins" color="15" fill="1" visible="yes" active="no"/>
+<layer number="25" name="tNames" color="7" fill="1" visible="yes" active="no"/>
+<layer number="26" name="bNames" color="7" fill="1" visible="yes" active="no"/>
+<layer number="27" name="tValues" color="7" fill="1" visible="yes" active="no"/>
+<layer number="28" name="bValues" color="7" fill="1" visible="yes" active="no"/>
 <layer number="29" name="tStop" color="7" fill="3" visible="no" active="no"/>
 <layer number="30" name="bStop" color="7" fill="6" visible="no" active="no"/>
@@
 <layer number="35" name="tGlue" color="7" fill="4" visible="no" active="no"/>
 <layer number="36" name="bGlue" color="7" fill="5" visible="no" active="no"/>
-<layer number="37" name="tTest" color="7" fill="1" visible="no" active="no"/>
-<layer number="38" name="bTest" color="7" fill="1" visible="no" active="no"/>
+<layer number="37" name="tTest" color="7" fill="1" visible="yes" active="no"/>
+<layer number="38" name="bTest" color="7" fill="1" visible="yes" active="no"/>
 <layer number="39" name="tKeepout" color="4" fill="11" visible="no" active="no"/>
 <layer number="40" name="bKeepout" color="1" fill="11" visible="no" active="no"/>
@@
 <layer number="44" name="Drills" color="7" fill="1" visible="no" active="no"/>
 <layer number="45" name="Holes" color="7" fill="1" visible="no" active="no"/>
-<layer number="46" name="Milling" color="3" fill="1" visible="no" active="no"/>
-<layer number="47" name="Measures" color="7" fill="1" visible="no" active="no"/>
-<layer number="48" name="Document" color="7" fill="1" visible="no" active="no"/>
-<layer number="49" name="Reference" color="7" fill="1" visible="no" active="no"/>
-<layer number="50" name="dxf" color="7" fill="1" visible="no" active="no"/>
-<layer number="51" name="tDocu" color="11" fill="7" visible="no" active="no"/>
-<layer number="52" name="bDocu" color="7" fill="1" visible="no" active="no"/>
-<layer number="53" name="tGND_GNDA" color="7" fill="9" visible="no" active="no"/>
-<layer number="54" name="bGND_GNDA" color="1" fill="9" visible="no" active="no"/>
-<layer number="56" name="wert" color="7" fill="1" visible="no" active="no"/>
-<layer number="57" name="tCAD" color="7" fill="1" visible="no" active="no"/>
-<layer number="59" name="tCarbon" color="7" fill="1" visible="no" active="no"/>
-<layer number="60" name="bCarbon" color="7" fill="1" visible="no" active="no"/>
+<layer number="46" name="Milling" color="3" fill="1" visible="yes" active="no"/>
+<layer number="47" name="Measures" color="7" fill="1" visible="yes" active="no"/>
+<layer number="48" name="Document" color="7" fill="1" visible="yes" active="no"/>
+<layer number="49" name="Reference" color="7" fill="1" visible="yes" active="no"/>
+<layer number="50" name="dxf" color="7" fill="1" visible="yes" active="no"/>
+<layer number="51" name="tDocu" color="11" fill="7" visible="yes" active="no"/>
+<layer number="52" name="bDocu" color="7" fill="1" visible="yes" active="no"/>
+<layer number="53" name="tGND_GNDA" color="7" fill="9" visible="yes" active="no"/>
+<layer number="54" name="bGND_GNDA" color="1" fill="9" visible="yes" active="no"/>
+<layer number="56" name="wert" color="7" fill="1" visible="yes" active="no"/>
+<layer number="57" name="tCAD" color="7" fill="1" visible="yes" active="no"/>
+<layer number="59" name="tCarbon" color="7" fill="1" visible="yes" active="no"/>
+<layer number="60" name="bCarbon" color="7" fill="1" visible="yes" active="no"/>
 <layer number="90" name="Modules" color="5" fill="1" visible="yes" active="yes"/>
 <layer number="91" name="Nets" color="2" fill="1" visible="yes" active="yes"/>
@@
 <part name="C7" library="SparkFun-Capacitors" deviceset="CAP" device="0603-CAP" value="10nF"/>
 <part name="GND-ISO14" library="SparkFun-Aesthetics" deviceset="GND-ISO" device=""/>
-<part name="D13" library="diode" deviceset="SCHOTTKY-DIODE" device="SMD"/>
+<part name="D13" library="gipi" deviceset="DIODE" device=""/>
 <part name="R17" library="SparkFun-Passives" deviceset="RESISTOR" device="0603-RES" value="1k"/>
 <part name="R18" library="SparkFun-Passives" deviceset="RESISTOR" device="0603-RES" value="1k"/>

Commit message: Fix board layout.
Done some rerouting.
Parts:
- R15: device SparkFun-Passives:RESISTOR1206 -> SparkFun-Passives:RESISTOR0603-RES
Changed lines of the file:
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@@
 <part name="S2" library="SparkFun-Retired" deviceset="TAC_SWITCH" device="SMD" value="BOOT"/>
 <part name="GND-ISO12" library="SparkFun-Aesthetics" deviceset="GND-ISO" device=""/>
-<part name="R15" library="SparkFun-Passives" deviceset="RESISTOR" device="1206" value="10k"/>
+<part name="R15" library="SparkFun-Passives" deviceset="RESISTOR" device="0603-RES" value="10k"/>
 <part name="R16" library="SparkFun-Passives" deviceset="RESISTOR" device="0603-RES" value="1k"/>
 <part name="LED1" library="SparkFun-LED" deviceset="LED" device="0603"/>

Commit message: Rework some traces.
Parts:
- renumbered LED1 to XS
Connections:
- removed net N$28: D10.C, R14.1, SJ1.2
- removed net N$42: C8.2, C9.2, D13.C, R17.2
- new net VBATT: C8.2, C9.2, D10.C, D13.C, R14.1, R17.2, SJ1.2
Changed lines of the file:
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@@
 <grid distance="0.1" unitdist="inch" unit="inch" style="lines" multiple="1" display="no" altdistance="0.01" altunitdist="inch" altunit="inch"/>
 <layers>
-<layer number="1" name="Top" color="4" fill="1" visible="yes" active="no"/>
-<layer number="16" name="Bottom" color="1" fill="1" visible="yes" active="no"/>
-<layer number="17" name="Pads" color="2" fill="1" visible="yes" active="no"/>
-<layer number="18" name="Vias" color="2" fill="1" visible="yes" active="no"/>
-<layer number="19" name="Unrouted" color="2" fill="1" visible="yes" active="no"/>
-<layer number="20" name="Dimension" color="15" fill="1" visible="yes" active="no"/>
-<layer number="21" name="tPlace" color="7" fill="1" visible="yes" active="no"/>
-<layer number="22" name="bPlace" color="15" fill="1" visible="yes" active="no"/>
-<layer number="23" name="tOrigins" color="15" fill="1" visible="yes" active="no"/>
-<layer number="24" name="bOrigins" color="15" fill="1" visible="yes" active="no"/>
-<layer number="25" name="tNames" color="7" fill="1" visible="yes" active="no"/>
-<layer number="26" name="bNames" color="7" fill="1" visible="yes" active="no"/>
-<layer number="27" name="tValues" color="7" fill="1" visible="yes" active="no"/>
-<layer number="28" name="bValues" color="7" fill="1" visible="yes" active="no"/>
+<layer number="1" name="Top" color="4" fill="1" visible="no" active="no"/>
+<layer number="16" name="Bottom" color="1" fill="1" visible="no" active="no"/>
+<layer number="17" name="Pads" color="2" fill="1" visible="no" active="no"/>
+<layer number="18" name="Vias" color="2" fill="1" visible="no" active="no"/>
+<layer number="19" name="Unrouted" color="2" fill="1" visible="no" active="no"/>
+<layer number="20" name="Dimension" color="15" fill="1" visible="no" active="no"/>
+<layer number="21" name="tPlace" color="7" fill="1" visible="no" active="no"/>
+<layer number="22" name="bPlace" color="15" fill="1" visible="no" active="no"/>
+<layer number="23" name="tOrigins" color="15" fill="1" visible="no" active="no"/>
+<layer number="24" name="bOrigins" color="15" fill="1" visible="no" active="no"/>
+<layer number="25" name="tNames" color="7" fill="1" visible="no" active="no"/>
+<layer number="26" name="bNames" color="7" fill="1" visible="no" active="no"/>
+<layer number="27" name="tValues" color="7" fill="1" visible="no" active="no"/>
+<layer number="28" name="bValues" color="7" fill="1" visible="no" active="no"/>
 <layer number="29" name="tStop" color="7" fill="3" visible="no" active="no"/>
 <layer number="30" name="bStop" color="7" fill="6" visible="no" active="no"/>
@@
 <layer number="35" name="tGlue" color="7" fill="4" visible="no" active="no"/>
 <layer number="36" name="bGlue" color="7" fill="5" visible="no" active="no"/>
-<layer number="37" name="tTest" color="7" fill="1" visible="yes" active="no"/>
-<layer number="38" name="bTest" color="7" fill="1" visible="yes" active="no"/>
+<layer number="37" name="tTest" color="7" fill="1" visible="no" active="no"/>
+<layer number="38" name="bTest" color="7" fill="1" visible="no" active="no"/>
 <layer number="39" name="tKeepout" color="4" fill="11" visible="no" active="no"/>
 <layer number="40" name="bKeepout" color="1" fill="11" visible="no" active="no"/>
@@
 <layer number="44" name="Drills" color="7" fill="1" visible="no" active="no"/>
 <layer number="45" name="Holes" color="7" fill="1" visible="no" active="no"/>
-<layer number="46" name="Milling" color="3" fill="1" visible="yes" active="no"/>
-<layer number="47" name="Measures" color="7" fill="1" visible="yes" active="no"/>
-<layer number="48" name="Document" color="7" fill="1" visible="yes" active="no"/>
-<layer number="49" name="Reference" color="7" fill="1" visible="yes" active="no"/>
-<layer number="50" name="dxf" color="7" fill="1" visible="yes" active="no"/>
-<layer number="51" name="tDocu" color="11" fill="7" visible="yes" active="no"/>
-<layer number="52" name="bDocu" color="7" fill="1" visible="yes" active="no"/>
-<layer number="53" name="tGND_GNDA" color="7" fill="9" visible="yes" active="no"/>
-<layer number="54" name="bGND_GNDA" color="1" fill="9" visible="yes" active="no"/>
-<layer number="56" name="wert" color="7" fill="1" visible="yes" active="no"/>
-<layer number="57" name="tCAD" color="7" fill="1" visible="yes" active="no"/>
-<layer number="59" name="tCarbon" color="7" fill="1" visible="yes" active="no"/>
-<layer number="60" name="bCarbon" color="7" fill="1" visible="yes" active="no"/>
+<layer number="46" name="Milling" color="3" fill="1" visible="no" active="no"/>
+<layer number="47" name="Measures" color="7" fill="1" visible="no" active="no"/>
+<layer number="48" name="Document" color="7" fill="1" visible="no" active="no"/>
+<layer number="49" name="Reference" color="7" fill="1" visible="no" active="no"/>
+<layer number="50" name="dxf" color="7" fill="1" visible="no" active="no"/>
+<layer number="51" name="tDocu" color="11" fill="7" visible="no" active="no"/>
+<layer number="52" name="bDocu" color="7" fill="1" visible="no" active="no"/>
+<layer number="53" name="tGND_GNDA" color="7" fill="9" visible="no" active="no"/>
+<layer number="54" name="bGND_GNDA" color="1" fill="9" visible="no" active="no"/>
+<layer number="56" name="wert" color="7" fill="1" visible="no" active="no"/>
+<layer number="57" name="tCAD" color="7" fill="1" visible="no" active="no"/>
+<layer number="59" name="tCarbon" color="7" fill="1" visible="no" active="no"/>
+<layer number="60" name="bCarbon" color="7" fill="1" visible="no" active="no"/>
 <layer number="90" name="Modules" color="5" fill="1" visible="yes" active="yes"/>
 <layer number="91" name="Nets" color="2" fill="1" visible="yes" active="yes"/>
@@
 <part name="R15" library="SparkFun-Passives" deviceset="RESISTOR" device="0603-RES" value="10k"/>
 <part name="R16" library="SparkFun-Passives" deviceset="RESISTOR" device="0603-RES" value="1k"/>
-<part name="LED1" library="SparkFun-LED" deviceset="LED" device="0603"/>
+<part name="XS" library="SparkFun-LED" deviceset="LED" device="0603"/>
 <part name="GND-ISO13" library="SparkFun-Aesthetics" deviceset="GND-ISO" device=""/>
 <part name="BOOST" library="SparkFun-PowerIC" deviceset="V_REG_TPS61040" device="SMD"/>
@@
 <instance part="R15" gate="G$1" x="-33.02" y="-12.7" rot="R270"/>
 <instance part="R16" gate="G$1" x="96.52" y="-119.38"/>
-<instance part="LED1" gate="G$1" x="109.22" y="-119.38" rot="R90"/>
+<instance part="XS" gate="G$1" x="109.22" y="-119.38" rot="R90"/>
 <instance part="GND-ISO13" gate="G$1" x="121.92" y="-129.54"/>
 <instance part="BOOST" gate="G$1" x="33.02" y="-220.98"/>
@@
 <segment>
 <pinref part="GND-ISO13" gate="G$1" pin="GND-ISO"/>
-<pinref part="LED1" gate="G$1" pin="C"/>
+<pinref part="XS" gate="G$1" pin="C"/>
 <wire x1="121.92" y1="-127" x2="121.92" y2="-119.38" width="0.1524" layer="91"/>
 <wire x1="121.92" y1="-119.38" x2="114.3" y2="-119.38" width="0.1524" layer="91"/>
@@
 </segment>
 </net>
-<net name="N$28" class="0">
-<segment>
-<pinref part="SJ1" gate="G$1" pin="2"/>
-<wire x1="-22.86" y1="88.9" x2="-30.48" y2="88.9" width="0.1524" layer="91"/>
-<pinref part="D10" gate="G$1" pin="C"/>
-<wire x1="-30.48" y1="76.2" x2="-30.48" y2="88.9" width="0.1524" layer="91"/>
-<junction x="-30.48" y="88.9"/>
-<pinref part="R14" gate="G$1" pin="1"/>
-<wire x1="-30.48" y1="88.9" x2="-30.48" y2="91.44" width="0.1524" layer="91"/>
-</segment>
-</net>
 <net name="N$32" class="0">
 <segment>
@@
 <segment>
 <pinref part="R16" gate="G$1" pin="2"/>
-<pinref part="LED1" gate="G$1" pin="A"/>
+<pinref part="XS" gate="G$1" pin="A"/>
 <wire x1="101.6" y1="-119.38" x2="106.68" y2="-119.38" width="0.1524" layer="91"/>
 </segment>
@@
 </segment>
 </net>
-<net name="N$42" class="0">
+<net name="VBATT" class="0">
 <segment>
 <pinref part="D13" gate="G$1" pin="C"/>
@@
 <wire x1="114.3" y1="-205.74" x2="114.3" y2="-223.52" width="0.1524" layer="91"/>
 <junction x="99.06" y="-205.74"/>
-</segment>
-</net>
+<wire x1="114.3" y1="-205.74" x2="124.46" y2="-205.74" width="0.1524" layer="91"/>
+<junction x="114.3" y="-205.74"/>
+<label x="124.46" y="-205.74" size="1.778" layer="95" xref="yes"/>
+</segment>
+<segment>
+<pinref part="SJ1" gate="G$1" pin="2"/>
+<wire x1="-22.86" y1="88.9" x2="-30.48" y2="88.9" width="0.1524" layer="91"/>
+<pinref part="D10" gate="G$1" pin="C"/>
+<wire x1="-30.48" y1="76.2" x2="-30.48" y2="88.9" width="0.1524" layer="91"/>
+<junction x="-30.48" y="88.9"/>
+<pinref part="R14" gate="G$1" pin="1"/>
+<wire x1="-30.48" y1="88.9" x2="-30.48" y2="91.44" width="0.1524" layer="91"/>
+<wire x1="-30.48" y1="88.9" x2="-38.1" y2="88.9" width="0.1524" layer="91"/>
+<label x="-38.1" y="88.9" size="1.778" layer="95" rot="R180" xref="yes"/>
+</segment>
+</net>

Commit message: Fix label mosfet.
Parts:
- renumbered NFET to N-FET
Changed lines of the file:
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@@
 <part name="GND-ISO2" library="SparkFun-Aesthetics" deviceset="GND-ISO" device=""/>
 <part name="JP6" library="SparkFun-Connectors" deviceset="M02" device="JST-PTH-VERT"/>
-<part name="NFET" library="GeekAmmo" deviceset="P-CHANNEL-MOSFET" device=""/>
+<part name="N-FET" library="GeekAmmo" deviceset="P-CHANNEL-MOSFET" device=""/>
 </parts>
 <sheets>
@@
 <instance part="GND-ISO2" gate="G$1" x="-33.02" y="20.32"/>
 <instance part="JP6" gate="G$1" x="-27.94" y="-208.28" rot="R270"/>
-<instance part="NFET" gate="G$1" x="-15.24" y="-220.98" rot="R90"/>
+<instance part="N-FET" gate="G$1" x="-15.24" y="-220.98" rot="R90"/>
 </instances>
 <busses>
@@
 <wire x1="-5.08" y1="-205.74" x2="10.16" y2="-205.74" width="0.1524" layer="91"/>
 <junction x="10.16" y="-205.74"/>
-<pinref part="NFET" gate="G$1" pin="D"/>
+<pinref part="N-FET" gate="G$1" pin="D"/>
 <wire x1="-7.62" y1="-218.44" x2="-5.08" y2="-218.44" width="0.1524" layer="91"/>
 </segment>
@@
 <wire x1="-17.78" y1="-241.3" x2="10.16" y2="-241.3" width="0.1524" layer="91"/>
 <wire x1="-25.4" y1="-215.9" x2="-25.4" y2="-241.3" width="0.1524" layer="91"/>
-<pinref part="NFET" gate="G$1" pin="G"/>
+<pinref part="N-FET" gate="G$1" pin="G"/>
 <wire x1="-17.78" y1="-226.06" x2="-17.78" y2="-241.3" width="0.1524" layer="91"/>
 <junction x="-17.78" y="-241.3"/>
@@
 <pinref part="JP6" gate="G$1" pin="1"/>
 <wire x1="-27.94" y1="-215.9" x2="-27.94" y2="-218.44" width="0.1524" layer="91"/>
-<pinref part="NFET" gate="G$1" pin="S"/>
+<pinref part="N-FET" gate="G$1" pin="S"/>
 <wire x1="-27.94" y1="-218.44" x2="-22.86" y2="-218.44" width="0.1524" layer="91"/>
 </segment>
